Commit message: Updated docs. Updated rviz model.

File: src/ros/src/ros_homebot_description/urdf/homebot.urdf.xacro (robot description, xacro)
@@ -1,19 +1,8 @@
-<?xml version="1.0"?>
-<robot name="homebot"
-    xmlns:xacro="http://www.ros.org/wiki/xacro">
-    <xacro:macro name="box_inertia" params="mass x y z">
-    	<inertia
-    		ixx="${mass*(y*y+z*z)/12}" ixy="0" ixz="0"
-			iyy="${mass*(x*x+z*z)/12}" iyz="0" izz="${mass*(x*x+z*z)/12}" />
-	</xacro:macro>
+<?xml version="1.0" encoding="UTF-8"?>
+<robot xmlns:xacro="http://www.ros.org/wiki/xacro" name="homebot">
     <xacro:include filename="$(find ros_homebot_description)/urdf/materials.urdf.xacro" />
-    <!-- width in meters -->
-    <property name="torso_x_size" value="0.1" />
-    <!-- length in meters -->
-    <property name="torso_y_size" value="0.205" />
-    <!-- height in meters -->
-    <property name="torso_z_size" value="0.03" />
-    <!-- torso mass (not including legs) in kg -->
-    <property name="torso_mass" value="0.920" />
+    <!-- dimensions in meters -->
+    <property name="torso_radius" value="0.075" />
+    <property name="torso_height" value="0.15" />
     <link name="base_footprint">
         <visual>
@@ -23,40 +12,42 @@
             </geometry>
         </visual>
-	    <inertial>
-			<mass value="0.0001" />
-			<origin xyz="0 0 0" />
-			<inertia
-				ixx="0.0001" ixy="0.0" ixz="0.0"
-			  	iyy="0.0001" iyz="0.0" izz="0.0001" />
-	    </inertial>
+        <inertial>
+            <mass value="0.0001" />
+            <origin xyz="0 0 0" />
+            <inertia ixx="0.0001" ixy="0.0" ixz="0.0" iyy="0.0001" iyz="0.0" izz="0.0001" />
+        </inertial>
     </link>
+    <link name="head">
+        <visual>
+            <geometry>
+                <sphere radius="${torso_radius}" />
+            </geometry>
+            <material name="white" />
+        </visual>
+    </link>
+    <link name="base_link">
+        <visual>
+            <geometry>
+                <cylinder length="${torso_height}" radius="${torso_radius}" />
+            </geometry>
+            <material name="blue">
+                <color rgba="0 0 .8 1" />
+            </material>
+        </visual>
+    </link>
+    <joint name="base_footprint_joint" type="fixed">
+        <origin xyz="0 0 0" rpy="0 0 0" />
+        <parent link="base_footprint" />
+        <child link="base_link" />
+    </joint>
+    <joint name="torso_head_joint" type="fixed">
+        <origin xyz="0 0 0" rpy="0 0 0" />
+        <parent link="base_link" />
+        <child link="head" />
+    </joint>
+    <!--
     <gazebo reference="base_footprint">
         <turnGravityOff>false</turnGravityOff>
     </gazebo>
-	<joint name="base_footprint_joint" type="fixed">
-		<origin xyz="0 0 ${total_leg_height}" rpy="0 0 0" />
-		<parent link="base_footprint"/>
-		<child link="base_link" />
-	</joint>
-    <link name="base_link">
-        <visual>
-            <geometry>
-                <box size="${torso_x_size} ${torso_y_size} ${torso_z_size}" />
-            </geometry>
-            <material name="red"/>
-        </visual>
-        <collision>
-            <geometry>
-                <box size="${torso_x_size} ${torso_y_size} ${torso_z_size}" />
-            </geometry>
-        </collision>
-	    <inertial>
-	        <origin xyz="0 0 0" rpy="0 0 0" />
-	        <mass value="${torso_mass}" />
-	        <xacro:box_inertia
-	            mass="${torso_mass}"
-	            x="${torso_x_size}" y="${torso_y_size}" z="${torso_z_size}" />
-	    </inertial>
-    </link>
     <gazebo reference="base_link">
         <material>Gazebo/Red</material>
@@ -68,3 +59,4 @@
         </plugin>
     </gazebo>
+    -->
 </robot>

Commit message: Updated links in urdf model.

File: src/ros/src/ros_homebot_description/urdf/homebot.urdf.xacro (robot description, xacro)
@@ -3,6 +3,8 @@
     <xacro:include filename="$(find ros_homebot_description)/urdf/materials.urdf.xacro" />
     <!-- dimensions in meters -->
-    <property name="torso_radius" value="0.075" />
-    <property name="torso_height" value="0.15" />
+    <property name="torso_radius" value="0.075" /><!-- 150 mm diameter = 75 mm radius -->
+    <property name="torso_height" value="0.16" /><!-- 160 mm height -->
+    <property name="camera_radius" value="0.008" />
+    <property name="camera_thickness" value="0.005" />
     <link name="base_footprint">
         <visual>
@@ -23,5 +25,15 @@
                 <sphere radius="${torso_radius}" />
             </geometry>
-            <material name="white" />
+            <origin xyz="0 0 0" rpy="0 0 0" />
+            <material name="blue" />
+        </visual>
+    </link>
+    <link name="camera">
+        <visual>
+            <geometry>
+                <cylinder length="${camera_thickness}" radius="${camera_radius}" />
+            </geometry>
+            <origin xyz="0 0 0" rpy="0 90 0" />
+            <material name="black" />
         </visual>
     </link>
@@ -31,18 +43,22 @@
                 <cylinder length="${torso_height}" radius="${torso_radius}" />
             </geometry>
-            <material name="blue">
-                <color rgba="0 0 .8 1" />
-            </material>
+            <origin xyz="0 0 ${torso_height/2}" rpy="0 0 0" />
+            <material name="red" />
         </visual>
     </link>
     <joint name="base_footprint_joint" type="fixed">
-        <origin xyz="0 0 0" rpy="0 0 0" />
         <parent link="base_footprint" />
         <child link="base_link" />
+        <origin xyz="0 0 0" rpy="0 0 0" />
     </joint>
     <joint name="torso_head_joint" type="fixed">
-        <origin xyz="0 0 0" rpy="0 0 0" />
         <parent link="base_link" />
         <child link="head" />
+        <origin xyz="0 0 ${torso_height+torso_radius}" rpy="0 0 0" />
+    </joint>
+    <joint name="head_camera_joint" type="fixed">
+        <parent link="head" />
+        <child link="camera" />
+        <origin xyz="0 ${torso_radius} 0" rpy="0 0 0" />
     </joint>
     <!--

Commit message: Added neck link. Fixed joints to be movable in rviz.

File: src/ros/src/ros_homebot_description/urdf/homebot.urdf.xacro (robot description, xacro)
@@ -5,6 +5,8 @@
     <property name="torso_radius" value="0.075" /><!-- 150 mm diameter = 75 mm radius -->
     <property name="torso_height" value="0.16" /><!-- 160 mm height -->
+    <property name="neck_height" value="0.015" />
     <property name="camera_radius" value="0.008" />
     <property name="camera_thickness" value="0.005" />
+    <property name="M_PI" value="3.141592653589793" />
     <link name="base_footprint">
         <visual>
@@ -19,4 +21,22 @@
             <inertia ixx="0.0001" ixy="0.0" ixz="0.0" iyy="0.0001" iyz="0.0" izz="0.0001" />
         </inertial>
+    </link>
+    <link name="base_link">
+        <visual>
+            <geometry>
+                <cylinder length="${torso_height}" radius="${torso_radius}" />
+            </geometry>
+            <origin xyz="0 0 ${torso_height/2}" rpy="0 0 0" />
+            <material name="red" />
+        </visual>
+    </link>
+    <link name="neck">
+        <visual>
+            <geometry>
+                <cylinder length="${neck_height}" radius="${torso_radius}" />
+            </geometry>
+            <origin xyz="0 0 ${neck_height/2}" rpy="0 0 0" />
+            <material name="green" />
+        </visual>
     </link>
     <link name="head">
@@ -38,24 +58,24 @@
         </visual>
     </link>
-    <link name="base_link">
-        <visual>
-            <geometry>
-                <cylinder length="${torso_height}" radius="${torso_radius}" />
-            </geometry>
-            <origin xyz="0 0 ${torso_height/2}" rpy="0 0 0" />
-            <material name="red" />
-        </visual>
-    </link>
-    <joint name="base_footprint_joint" type="fixed">
+    <joint name="footprint_to_base_link_joint" type="fixed">
         <parent link="base_footprint" />
         <child link="base_link" />
         <origin xyz="0 0 0" rpy="0 0 0" />
     </joint>
-    <joint name="torso_head_joint" type="fixed">
+    <joint name="base_link_to_neck_joint" type="continuous">
         <parent link="base_link" />
+        <child link="neck" />
+        <origin xyz="0 0 ${torso_height}" rpy="0 0 0" />
+        <axis xyz="0 0 1" />
+    </joint>
+    <joint name="neck_to_head_joint" type="revolute">
+        <parent link="neck" />
         <child link="head" />
-        <origin xyz="0 0 ${torso_height+torso_radius}" rpy="0 0 0" />
+        <origin xyz="0 0 ${neck_height+torso_radius}" rpy="${M_PI/2} 0 0" />
+        <axis xyz="1 0 0" />
+        <!-- Should match TILT_MIN/TILT_MAX in ros_homebot_python/constants.py -->
+        <limit lower="${(90-65)*M_PI/180}" upper="${(90+65)*M_PI/180}" effort="50" velocity="1"/>
     </joint>
-    <joint name="head_camera_joint" type="fixed">
+    <joint name="head_to_camera_joint" type="fixed">
         <parent link="head" />
         <child link="camera" />

Commit message: Refactored urdf model. Modified head node to periodically publish joint states.

File: src/ros/src/ros_homebot_description/urdf/homebot.urdf.xacro (robot description, xacro)
@@ -66,5 +66,5 @@
         <parent link="base_link" />
         <child link="neck" />
-        <origin xyz="0 0 ${torso_height}" rpy="0 0 0" />
+        <origin xyz="0 0 ${torso_height+neck_height}" rpy="0 ${M_PI} 0" />
         <axis xyz="0 0 1" />
     </joint>
@@ -72,5 +72,5 @@
         <parent link="neck" />
         <child link="head" />
-        <origin xyz="0 0 ${neck_height+torso_radius}" rpy="${M_PI/2} 0 0" />
+        <origin xyz="0 0 ${-(torso_radius)}" rpy="${M_PI/2} 0 ${M_PI}" />
         <axis xyz="1 0 0" />
         <!-- Should match TILT_MIN/TILT_MAX in ros_homebot_python/constants.py -->

Commit message: Fixed xacro warnings.

File: src/ros/src/ros_homebot_description/urdf/homebot.urdf.xacro (robot description, xacro)
@@ -3,10 +3,10 @@
     <xacro:include filename="$(find ros_homebot_description)/urdf/materials.urdf.xacro" />
     <!-- dimensions in meters -->
-    <property name="torso_radius" value="0.075" /><!-- 150 mm diameter = 75 mm radius -->
-    <property name="torso_height" value="0.16" /><!-- 160 mm height -->
-    <property name="neck_height" value="0.015" />
-    <property name="camera_radius" value="0.008" />
-    <property name="camera_thickness" value="0.005" />
-    <property name="M_PI" value="3.141592653589793" />
+    <xacro:property name="torso_radius" value="0.075" /><!-- 150 mm diameter = 75 mm radius -->
+    <xacro:property name="torso_height" value="0.16" /><!-- 160 mm height -->
+    <xacro:property name="neck_height" value="0.015" />
+    <xacro:property name="camera_radius" value="0.008" />
+    <xacro:property name="camera_thickness" value="0.005" />
+    <xacro:property name="M_PI" value="3.141592653589793" />
     <link name="base_footprint">
         <visual>

Commit message: Added 18650 based 3rd generation battery pack. Added recharge dock. Added PID controller for head pan motor.

File: src/ros/src/ros_homebot_description/urdf/homebot.urdf.xacro (robot description, xacro)
@@ -1,3 +1,6 @@
 <?xml version="1.0" encoding="UTF-8"?>
+<!--
+This is loaded by robot_state_publisher and used to calculate poses from odometry and joint messages.
+-->
 <robot xmlns:xacro="http://www.ros.org/wiki/xacro" name="homebot">
     <xacro:include filename="$(find ros_homebot_description)/urdf/materials.urdf.xacro" />
@@ -31,4 +34,13 @@
             <origin xyz="0 0 ${torso_height/2}" rpy="0 0 0" />
             <material name="red" />
+        </visual>
+    </link>
+    <link name="imu">
+        <visual>
+            <geometry>
+                <box size=".03 .015 .01" />
+            </geometry>
+            <origin xyz="0 0 0" rpy="0 0 0" />
+            <material name="orange" />
         </visual>
     </link>
@@ -71,5 +83,11 @@
         <child link="neck" />
         <origin xyz="0 0 ${torso_height+neck_height}" rpy="0 ${M_PI} 0" />
+        <!--<origin xyz="0 0 ${torso_height}" rpy="0 ${M_PI} 0" />-->
         <axis xyz="0 0 1" />
+    </joint>
+    <joint name="base_link_to_imu" type="fixed">
+        <parent link="base_link" />
+        <child link="imu" />
+        <origin xyz="0 ${torso_radius - .015} ${torso_height - .01}" rpy="0 0 0" />
     </joint>
     <joint name="neck_to_head_joint" type="revolute">
